Commit message: Fixed gazebo and updated xacro

File: src/ball_bot_pde4430/urdf/ball_bot.xacro (robot description, xacro)
@@ -1,16 +1,16 @@
 <?xml version="1.0"?>
 <robot name="ball_bot" xmlns:xacro="http://www.ros.org/wiki/xacro">
-  <!-- ========================== -->
-  <!-- XACRO PROPERTIES -->
-  <!-- ========================== -->
-  <xacro:property name="base_length" value="0.25"/>
+  <!-- ========================================================= -->
+  <!-- PARAMETERS -->
+  <!-- ========================================================= -->
+  <xacro:property name="base_length" value="0.30"/>
   <xacro:property name="base_width"  value="0.25"/>
   <xacro:property name="base_height" value="0.10"/>
   <xacro:property name="wheel_radius" value="0.04"/>
-  <xacro:property name="wheel_width"  value="0.03"/>
+  <xacro:property name="wheel_width"  value="0.02"/>
   <xacro:property name="caster_radius" value="0.025"/>
   <xacro:property name="finger_length" value="0.12"/>
   <xacro:property name="finger_width"  value="0.02"/>
-  <xacro:property name="finger_height" value="0.06"/>
+  <xacro:property name="finger_height" value="0.08"/>
   <xacro:property name="lidar_radius" value="0.05"/>
   <xacro:property name="lidar_height" value="0.02"/>
@@ -18,8 +18,8 @@
   <material name="green"><color rgba="0 1 0 1"/></material>
   <material name="black"><color rgba="0 0 0 1"/></material>
-  <material name="grey"><color rgba="0.7 0.7 0.7 1"/></material>
-  <!-- ========================== -->
+  <material name="grey"><color rgba="0.6 0.6 0.6 1"/></material>
+  <!-- ========================================================= -->
   <!-- BASE LINK -->
-  <!-- ========================== -->
+  <!-- ========================================================= -->
   <link name="base_link">
     <visual>
@@ -39,15 +39,15 @@
       <mass value="1.0"/>
       <origin xyz="0 0 ${base_height/2}"/>
-      <inertia ixx="0.02" iyy="0.02" izz="0.02"
-               ixy="0" ixz="0" iyz="0"/>
+      <inertia ixx="0.02" ixy="0" ixz="0"
+               iyy="0.02" iyz="0" izz="0.02"/>
     </inertial>
   </link>
-  <!-- ========================== -->
+  <!-- ========================================================= -->
   <!-- WHEEL MACRO -->
-  <!-- ========================== -->
+  <!-- ========================================================= -->
   <xacro:macro name="wheel" params="name x y">
     <link name="${name}">
       <visual>
-        <origin xyz="0 0 0" rpy="1.5708 0 0"/>
+        <origin rpy="0 1.5708 0"/>
         <geometry>
           <cylinder radius="${wheel_radius}" length="${wheel_width}"/>
@@ -56,5 +56,5 @@
       </visual>
       <collision>
-        <origin xyz="0 0 0" rpy="1.5708 0 0"/>
+        <origin rpy="0 1.5708 0"/>
         <geometry>
           <cylinder radius="${wheel_radius}" length="${wheel_width}"/>
@@ -64,6 +64,6 @@
         <mass value="0.1"/>
         <origin xyz="0 0 0"/>
-        <inertia ixx="0.00016" iyy="0.00016" izz="0.00016"
-                 ixy="0" ixz="0" iyz="0"/>
+        <inertia ixx="0.0001" ixy="0" ixz="0"
+                 iyy="0.0001" iyz="0" izz="0.0001"/>
       </inertial>
     </link>
@@ -75,11 +75,11 @@
     </joint>
   </xacro:macro>
-  <!-- Instantiate wheels -->
-  <xacro:wheel name="rear_left_wheel"  x="-0.05" y="0.12"/>
-  <xacro:wheel name="rear_right_wheel" x="-0.05" y="-0.12"/>
-  <!-- ========================== -->
-  <!-- FRONT CASTER -->
-  <!-- ========================== -->
-  <link name="front_caster">
+  <!-- Rear wheels -->
+  <xacro:wheel name="rear_left_wheel"  x="-0.10" y="0.12"/>
+  <xacro:wheel name="rear_right_wheel" x="-0.10" y="-0.12"/>
+  <!-- ========================================================= -->
+  <!-- CENTER CASTER WHEEL (ball-like support) -->
+  <!-- ========================================================= -->
+  <link name="caster_wheel">
     <visual>
       <geometry><sphere radius="${caster_radius}"/></geometry>
@@ -92,35 +92,63 @@
       <mass value="0.05"/>
       <origin xyz="0 0 0"/>
-      <inertia ixx="0.000009" iyy="0.000009" izz="0.000009"
-               ixy="0" ixz="0" iyz="0"/>
+      <inertia ixx="0.00001" ixy="0" ixz="0"
+               iyy="0.00001" iyz="0" izz="0.00001"/>
     </inertial>
   </link>
-  <joint name="front_caster_joint" type="fixed">
+  <joint name="caster_joint" type="fixed">
     <parent link="base_link"/>
-    <child link="front_caster"/>
-    <origin xyz="0.09 0 ${caster_radius}"/>
+    <child link="caster_wheel"/>
+    <origin xyz="0.10 0 ${caster_radius}"/>
   </joint>
-  <!-- ========================== -->
+  <!-- ========================================================= -->
+  <!-- LEFT + RIGHT GRIPPER FINGERS -->
+  <!-- ========================================================= -->
+  <link name="left_finger">
+    <visual>
+      <geometry>
+        <box size="${finger_length} ${finger_width} ${finger_height}"/>
+      </geometry>
+      <material name="grey"/>
+    </visual>
+  </link>
+  <link name="right_finger">
+    <visual>
+      <geometry>
+        <box size="${finger_length} ${finger_width} ${finger_height}"/>
+      </geometry>
+      <material name="grey"/>
+    </visual>
+  </link>
+  <!-- Joints for the gripper fingers -->
+  <joint name="left_finger_joint" type="revolute">
+    <parent link="base_link"/>
+    <child link="left_finger"/>
+    <origin xyz="0.15 0.06 0.06"/>
+    <axis xyz="0 0 1"/>
+    <limit lower="-0.5" upper="0.5" effort="10" velocity="1.0"/>
+  </joint>
+  <joint name="right_finger_joint" type="revolute">
+    <parent link="base_link"/>
+    <child link="right_finger"/>
+    <origin xyz="0.15 -0.06 0.06"/>
+    <axis xyz="0 0 -1"/>
+    <limit lower="-0.5" upper="0.5" effort="10" velocity="1.0"/>
+  </joint>
+  <!-- ========================================================= -->
   <!-- LIDAR -->
-  <!-- ========================== -->
+  <!-- ========================================================= -->
   <link name="lidar_link">
     <visual>
-      <geometry><cylinder radius="${lidar_radius}" length="${lidar_height}"/></geometry>
+      <origin xyz="0 0 0"/>
+      <geometry>
+        <cylinder radius="${lidar_radius}" length="${lidar_height}"/>
+      </geometry>
       <material name="black"/>
     </visual>
-    <collision>
-      <geometry><cylinder radius="0.03" length="${lidar_height}"/></geometry>
-    </collision>
-    <inertial>
-      <mass value="0.05"/>
-      <origin xyz="0 0 0"/>
-      <inertia ixx="0.000005" iyy="0.000005" izz="0.000008"
-               ixy="0" ixz="0" iyz="0"/>
-    </inertial>
   </link>
   <joint name="lidar_joint" type="fixed">
     <parent link="base_link"/>
     <child link="lidar_link"/>
-    <origin xyz="0 0 0.10"/>
+    <origin xyz="0 0 0.15"/>
   </joint>
 </robot>
